File: PCB/Kicad/memory_controller/memory_controller.kicad_sch (KiCad schematic)
At the start: 34 parts

Commit message: bus in progress
Connections:
- net GND: no longer Rd1.2, Rd10.2, Rd2.2, Rd5.2, Rd6.2, Rd7.2
- net VCC: now also Dd1.2 (A), Dd10.2 (A), Dd2.2 (A), Dd5.2 (A), Dd6.2 (A), Dd7.2 (A)
- net ~{OE}_MUX_n: now also Rd6.2; no longer Dd6.2 (A)
- net ~{OE}_n: now also Rd10.2, Rd2.2; no longer Dd10.2 (A), Dd2.2 (A)
- net ~{OE}_p: now also Rd1.2; no longer Dd1.2 (A)
- net ~{OUTPUT_ENABLE}: now also Rd7.2; no longer Dd7.2 (A)
- net ~{WE}_mem: now also Rd5.2; no longer Dd5.2 (A)
