File: PCB/Kicad/memory_controller/memory_controller.kicad_pcb (KiCad board)
At the start: 6 copper layers, 180 x 100 mm, 116 parts, among them U1 74245, U10 74283, U11 74377, U12 74377, U13 74245, U14 74245, U15 74245, U16 74245, U17 74245, U18 74245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

Commit message: decoupling C RAM ROM
Parts:
- added C26: 100nF, Capacitor_SMD:C_0402_1005Metric, F.Cu at (161.1, 101.6)
- added C27: 100nF, Capacitor_SMD:C_0402_1005Metric, F.Cu at (150.1, 84.2)
- added C28: 100nF, Capacitor_SMD:C_0402_1005Metric, F.Cu at (150.1, 123.3)
Routing:
- net GND: track 169.1 -> 172.5 mm, vias 86 -> 89
- net VCC: track 13.0 -> 11.2 mm, vias 3 -> 2
