File: PCB/Kicad/control_unit/control_unit.kicad_pcb (KiCad board)
At the start: 6 copper layers, 150 x 150 mm, 348 parts, among them J1 in, J2 in, J3 in, J4 in, J5 in, J6 in, J7 in, J8 in, SW1 SW_Push, U4 7408, U57 744067

Commit message: power schemat and layout
Parts:
- added C15: 120uF, mALUch_lib:16SVF1000M, B.Cu at (37.9, 117.7)
- added C16: 100nF, Capacitor_SMD:C_0402_1005Metric_Pad0.74x0.62mm_HandSolder, B.Cu at (58.5, 118.2)
- added C17: 15nF, Resistor_SMD:R_0402_1005Metric_Pad0.72x0.64mm_HandSolder, B.Cu at (80.2, 124.8)
- added C18: 1uF, Resistor_SMD:R_0402_1005Metric_Pad0.72x0.64mm_HandSolder, B.Cu at (77.5, 120.3)
- added C19: 470nF, Resistor_SMD:R_0402_1005Metric_Pad0.72x0.64mm_HandSolder, B.Cu at (71.2, 117.5)
- added C20: 430pF, Resistor_SMD:R_0402_1005Metric_Pad0.72x0.64mm_HandSolder, B.Cu at (81.0, 121.0)
- added C21: 150uF, mALUch_lib:16SVF1000M, B.Cu at (99.1, 119.5)
- added C22: 120uF, mALUch_lib:16SVF1000M, B.Cu at (50.3, 117.7)
- added IC1: LM3150MH_NOPB, mALUch_lib:SOP65P640X110-15L, B.Cu at (75.2, 123.5)
- added J9: Barrel_Jack_MountingPin, Connector_BarrelJack:BarrelJack_Horizontal, F.Cu at (23.0, 49.6)
- added L1: 3.3u, mALUch_lib:MLC1260, B.Cu at (80.7, 107.7)
- added M1: CSD17308Q3, mALUch_lib:CSD17308Q3, B.Cu at (66.1, 116.6)
- added M2: CSD18531Q5A, mALUch_lib:Q5A, B.Cu at (74.8, 115.3)
- added R1: 182kOhm, Resistor_SMD:R_0402_1005Metric_Pad0.72x0.64mm_HandSolder, B.Cu at (81.7, 124.8)
- added R2: 1.21kOhm, Resistor_SMD:R_0402_1005Metric_Pad0.72x0.64mm_HandSolder, B.Cu at (69.1, 117.5)
- added R3: 73.2kOhm, Resistor_SMD:R_0402_1005Metric_Pad0.72x0.64mm_HandSolder, B.Cu at (82.5, 121.0)
- added R4: 10kOhm, Resistor_SMD:R_0402_1005Metric_Pad0.72x0.64mm_HandSolder, B.Cu at (84.0, 122.2)
Routing:
- net /Power/VIN: track 0.00 -> 28.7 mm, vias 0 -> 3
- net GND: track 43.0 -> 56.0 mm, vias 38 -> 42
- net /Power/HG: track 0.00 -> 10.0 mm, vias 0 -> 2
- net /Power/SW: track 0.00 -> 9.95 mm
- net /Power/ILIM: track 0.00 -> 9.81 mm
- net /Power/LG: track 0.00 -> 7.78 mm, vias 0 -> 2
- net /Power/BST: track 0.00 -> 6.89 mm
- net /Power/FB: track 0.00 -> 6.71 mm
- net /Power/RON: track 0.00 -> 5.18 mm
- net /Power/SS: track 0.00 -> 2.53 mm
- net /Power/ICVCC: track 0.00 -> 1.45 mm
- added copper zone on B.Cu, net /Power/SW
- added copper zone on B.Cu, net GND
- added copper zone on B.Cu, net VCC
