File: PCB/Kicad/control_unit/control_unit.kicad_sch (KiCad schematic)
At the start: 14 parts, among them J1 in, J2 in, J3 in, J4 in, J5 in, J6 in, J7 in, J8 in

Commit message: power schemat and layout
Other:
- added sheet Power (power.kicad_sch)
Changed lines of the file:
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@@
+	)
+	(sheet
+		(at 38.1 152.4)
+		(size 25.4 12.7)
+		(exclude_from_sim no)
+		(in_bom yes)
+		(on_board yes)
+		(dnp no)
+		(fields_autoplaced yes)
+		(stroke
+			(width 0.1524)
+			(type solid)
+		)
+		(fill
+			(color 0 0 0 0)
+		)
+		(property "Sheetname" "Power"
+			(at 38.1 151.6884 0)
+			(show_name no)
+			(do_not_autoplace no)
+			(effects
+				(font
+					(size 1.27 1.27)
+				)
+				(justify left bottom)
+			)
+		)
+		(property "Sheetfile" "power.kicad_sch"
+			(at 38.1 165.6846 0)
+			(show_name no)
+			(do_not_autoplace no)
+			(effects
+				(font
+					(size 1.27 1.27)
+				)
+				(justify left top)
+			)
+		)
+		(instances
+			(project "control_unit"
+				(path "/dccec861-b967-466c-843e-d6d1ad6064ce"
+					(page "33")
+				)
+			)
+		)
 	)
 	(sheet
